File: Circuit_Through_Hole/fakeTecv5.kicad_pcb (KiCad board)
At the start: 2 copper layers, 25.4 x 52.1 mm, 33 parts, among them J1 EXTRA, J12 FET2 3,3, J14 GPS Pins, J16 Encoder Pads, J2 Conn_01x04_Socket, J38 JST-SH-4, J46 Conn_01x02_Socket, J5 I2C Oled screen, J50 JST-SH-4, J7 FET2 Drain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

Commit message: hw: refinement to roTecTH
Parts:
- added J3: FET2 Drain, faketec:SMD_PAD_1x01, B.Cu at (109.2, 65.0)
- added J4: FET2 3,3, faketec:SMD_PAD_1x01, B.Cu at (107.2, 64.9)
- moved J50 3.77 mm to (110.0, 60.5), turned to -90 degrees
- moved R5 3.60 mm to (101.0, 61.6)
- moved J12 1.85 mm to (109.3, 69.4)
- moved J7 1.54 mm to (111.4, 69.3)
- moved Q1 0.73 mm to (113.2, 66.2)
- moved R1 0.73 mm to (116.9, 66.2)
- moved R2 0.67 mm to (116.9, 70.9)
- moved Q2 0.67 mm to (113.2, 70.8)
- moved Q3 0.23 mm to (113.1, 75.3)
- moved BZ1 0.23 mm to (108.1, 74.0)
- moved R3 0.23 mm to (116.9, 75.3)
Routing:
- net /ENC_PUSH: track 22.9 -> 32.2 mm, vias 2 -> 4
- net /ENC_B: track 22.9 -> 31.0 mm
- net +3.3V: track 109.5 -> 116.3 mm
- net /ENC_A: track 21.2 -> 25.6 mm
- net /GPS_GND: track 12.4 -> 16.1 mm
- net GND: track 46.9 -> 43.6 mm, vias 35 -> 37
- net /Batt%: track 6.85 -> 9.07 mm
- net /VIBRATION: track 2.59 -> 1.63 mm
- net /BTN: track 21.8 -> 21.0 mm
Other:
- board text added: "10KΩ"
- board text added: "5020"
- board text added: "BUZ"
- board text added: "ROTARY> ENCODER"
- board text added: "charge <boost 300mA"
- board text added: "nchnFET"
- board text removed: "<ROTARY ENCODER"
