File: Circuit_Through_Hole/fakeTecv5.kicad_sch (KiCad schematic)
At the start: 36 parts, among them J1 EXTRA, J11 FET1 3,3, J12 FET2 3,3, J13 FET3 3,3, J14 GPS Pins, J16 Encoder Pads, J2 Conn_01x04_Socket, J38 JST-SH-4, J46 Conn_01x02_Socket, J5 I2C Oled screen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

Commit message: Update schematic and readme
Parts:
- removed J11: FET1 3,3, faketec:SMD_PAD_1x01, symbol Connector:Conn_01x01_Socket
- removed J13: FET3 3,3, faketec:SMD_PAD_1x01, symbol Connector:Conn_01x01_Socket
- removed J51: JST-SH-4, Connector_JST:JST_SH_SM04B-SRSS-TB_1x04-1MP_P1.00mm_Horizontal, symbol Connector_Generic_MountingPin:Conn_01x04_MountingPin
- removed J6: FET1 Drain, faketec:SMD_PAD_1x01, symbol Connector:Conn_01x01_Socket
- removed J8: FET3 Drain, faketec:SMD_PAD_1x01, symbol Connector:Conn_01x01_Socket
Other:
- note removed: "Socket Option"

Commit message: hw: refinement to roTecTH
Parts:
- added J3: FET2 Drain, faketec:SMD_PAD_1x01, symbol Connector:Conn_01x01_Socket
- added J4: FET2 3,3, faketec:SMD_PAD_1x01, symbol Connector:Conn_01x01_Socket
Connections:
- net +3.3V: now also J4.1 (Pin_1)
- net GPS_GND: now also J3.1 (Pin_1)
Changed lines of the file:
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@@
 	)
 	(junction
+		(at 240.03 58.42)
+		(diameter 0)
+		(color 0 0 0 0)
+	)
+	(junction
 		(at 72.39 33.02)
 		(diameter 0)
@@
 	(wire
 		(pts
+			(xy 257.81 67.31) (xy 257.81 64.77)
+		)
+		(stroke
+			(width 0)
+			(type default)
+		)
+	)
+	(wire
+		(pts
 			(xy 134.62 64.77) (xy 134.62 67.31)
 		)
@@
 	(wire
 		(pts
+			(xy 257.81 67.31) (xy 265.43 67.31)
+		)
+		(stroke
+			(width 0)
+			(type default)
+		)
+	)
+	(wire
+		(pts
 			(xy 240.03 58.42) (xy 240.03 63.5)
 		)
@@
 		)
 	)
+	(wire
+		(pts
+			(xy 240.03 58.42) (xy 265.43 58.42)
+		)
+		(stroke
+			(width 0)
+			(type default)
+		)
+	)
 	(image
 		(at 64.77 140.97)
@@
 	)
 	(symbol
+		(lib_id "Connector:Conn_01x01_Socket")
+		(at 270.51 67.31 0)
+		(unit 1)
+		(exclude_from_sim no)
+		(in_bom no)
+		(on_board yes)
+		(dnp no)
+		(fields_autoplaced yes)
+		(property "Reference" "J4"
+			(at 271.78 66.0399 0)
+			(effects
+				(font
+					(size 1.27 1.27)
+				)
+				(justify left)
+			)
+		)
+		(property "Value" "FET2 3,3"
+			(at 271.78 68.5799 0)
+			(effects
+				(font
+					(size 1.27 1.27)
+				)
+				(justify left)
+			)
+		)
+		(property "Footprint" "faketec:SMD_PAD_1x01"
+			(at 270.51 67.31 0)
+			(effects
+				(font
+					(size 1.27 1.27)
+				)
+				(hide yes)
+			)
+		)
+		(property "Datasheet" "~"
+			(at 270.51 67.31 0)
+			(effects
+				(font
+					(size 1.27 1.27)
+				)
+				(hide yes)
+			)
+		)
+		(property "Description" "Generic connector, single row, 01x01, script generated"
+			(at 270.51 67.31 0)
+			(effects
+				(font
+					(size 1.27 1.27)
+				)
+				(hide yes)
+			)
+		)
+		(pin "1"
+		)
+		(instances
+			(project "fakeTecv5"
+				(path "/9f57df6b-a9d3-4597-bf34-a2cbfc394ff5"
+					(reference "J4")
+					(unit 1)
+				)
+			)
+		)
+	)
+	(symbol
 		(lib_id "Device:R")
 		(at 162.56 139.7 90)
@@
 	)
 	(symbol
+		(lib_id "Connector:Conn_01x01_Socket")
+		(at 270.51 58.42 0)
+		(unit 1)
+		(exclude_from_sim no)
+		(in_bom no)
+		(on_board yes)
+		(dnp no)
+		(property "Reference" "J3"
+			(at 271.78 57.1499 0)
+			(effects
+				(font
+					(size 1.27 1.27)
+				)
+				(justify left)
+			)
+		)
+		(property "Value" "FET2 Drain"
+			(at 271.78 59.182 0)
+			(effects
+				(font
+					(size 1.27 1.27)
+				)
+				(justify left)
+			)
+		)
+		(property "Footprint" "faketec:SMD_PAD_1x01"
+			(at 270.51 58.42 0)
+			(effects
+				(font
+					(size 1.27 1.27)
+				)
+				(hide yes)
+			)
+		)
+		(property "Datasheet" "~"
+			(at 270.51 58.42 0)
+			(effects
+				(font
+					(size 1.27 1.27)
+				)
+				(hide yes)
+			)
+		)
+		(property "Description" "Generic connector, single row, 01x01, script generated"
+			(at 270.51 58.42 0)
+			(effects
+				(font
+					(size 1.27 1.27)
+				)
+				(hide yes)
+			)
+		)
+		(pin "1"
+		)
+		(instances
+			(project "fakeTecv5"
+				(path "/9f57df6b-a9d3-4597-bf34-a2cbfc394ff5"
+					(reference "J3")
+					(unit 1)
+				)
+			)
+		)
+	)
+	(symbol
 		(lib_id "power:+3.3V")
 		(at 149.86 26.67 0)
@@
 					(unit 1)
 				)
+			)
+		)
+	)
+	(symbol
+		(lib_id "power:+3.3V")
+		(at 257.81 64.77 0)
+		(unit 1)
+		(exclude_from_sim no)
+		(in_bom yes)
+		(on_board yes)
+		(dnp no)
+		(property "Reference" "#PWR025"
+			(at 257.81 68.58 0)
+			(effects
+				(font
+					(size 1.27 1.27)
+				)
+				(hide yes)
+			)
+		)
+		(property "Value" "+3.3V"
+			(at 257.81 60.96 0)
+			(effects
+				(font
+					(size 1.27 1.27)
+				)
+			)
+		)
+		(property "Footprint" ""
+			(at 257.81 64.77 0)
+			(effects
+				(font
+					(size 1.27 1.27)
+				)
+				(hide yes)
+			)
+		)
+		(property "Datasheet" ""
+			(at 257.81 64.77 0)
+			(effects
+				(font
+					(size 1.27 1.27)
+				)
+				(hide yes)
+			)
+		)
+		(property "Description" "Power symbol creates a global label with name \"+3.3V\""
+			(at 257.81 64.77 0)
+			(effects
+				(font
+					(size 1.27 1.27)
+				)
+				(hide yes)
+			)
+		)
+		(pin "1"
+		)
+		(instances
+			(project "fakeTecv5"
+				(path "/9f57df6b-a9d3-4597-bf34-a2cbfc394ff5"
+					(reference "#PWR025")
+					(unit 1)
+				)
